Commit message: Minor changes

File: Assets/Graphics/URDF/description/robot.urdf (robot description, URDF)
Before this commit: robot robot, 13 links, 12 joints
Links:
- added link camera, mass 0.05; collision mesh filename=package://fonbot_package/models/camera.dae scale=0.017 0.017 0.017; visual mesh filename=package://fonbot_package/models/camera.dae scale=0.017 0.017 0.017
- added link microphone, mass 0.05; collision mesh filename=package://fonbot_package/models/microphone.stl scale=0.008 0.008 0.008; visual mesh filename=package://fonbot_package/models/microphone.stl scale=0.008 0.008 0.008
- added link ultrasonic_back; collision mesh filename=package://fonbot_package/models/ultrasonic.dae scale=0.3 0.3 0.3; visual mesh filename=package://fonbot_package/models/ultrasonic.dae scale=0.3 0.3 0.3
- added link ultrasonic_bottom_back; collision mesh filename=package://fonbot_package/models/ultrasonic.dae scale=0.3 0.3 0.3; visual mesh filename=package://fonbot_package/models/ultrasonic.dae scale=0.3 0.3 0.3
- added link ultrasonic_bottom_front; collision mesh filename=package://fonbot_package/models/ultrasonic.dae scale=0.3 0.3 0.3; visual mesh filename=package://fonbot_package/models/ultrasonic.dae scale=0.3 0.3 0.3
- link ultrasonic_front: mass 0.05 -> None; geometry collision mesh filename=package://fonbot_package/models/ultrasonic.dae scale=0.3 0.3 0.3; visual mesh filename=package://fonbot_package/models/ultrasonic.dae scale=0.3 0.3 0.3
Joints:
- added joint camera_joint: type fixed, parent head, child camera
- added joint microphone_joint: type fixed, parent head, child microphone
- added joint ultrasonic_back_joint: type fixed, parent chassis, child ultrasonic_back, origin xyz=0 0.205 0.125
- added joint ultrasonic_bottom_back_joint: type fixed, parent chassis, child ultrasonic_bottom_back, origin xyz=0 0.205 0.125
- added joint ultrasonic_bottom_front_joint: type fixed, parent chassis, child ultrasonic_bottom_front, origin xyz=0 0.205 0.125
